Commit message: Add files via upload

File: robot_arm/urdf/mybot.urdf (robot description, URDF)
Before this commit: robot arm, 6 links, 5 joints
Links:
- added link left_gripper_base, mass 0.01; collision box size=0.005 0.005 0.02; visual box size=0.005 0.005 0.02
- added link left_gripper_finger, mass 0.01; collision box size=0.008 0.008 0.05; visual box size=0.008 0.008 0.05
- added link right_gripper_base, mass 0.01; collision box size=0.005 0.005 0.02; visual box size=0.005 0.005 0.02
- added link right_gripper_finger, mass 0.01; collision box size=0.005 0.005 0.05; visual box size=0.008 0.008 0.05
Joints:
- added joint l_g_base: type revolute, parent hand, child left_gripper_base, origin xyz=0 0.02 0.035 rpy=-0.9162 0 0, axis 1 0 0, limit lower=0 upper=0.5236 effort=30.0 velocity=1.0
- added joint l_g_finger: type fixed, parent left_gripper_base, child left_gripper_finger, origin xyz=0 -0.01 0.03 rpy=0.3926 0 0
- added joint r_g_base: type revolute, parent hand, child right_gripper_base, origin xyz=0 -0.02 0.035 rpy=0.9162 0 0, axis 1 0 0, limit lower=-0.5236 upper=0 effort=100.0 velocity=1.0
- added joint r_g_finger: type fixed, parent right_gripper_base, child right_gripper_finger, origin xyz=0 0.01 0.03 rpy=-0.3926 0 0

Commit message: Add files via upload

File: robot_arm/urdf/mybot.urdf (robot description, URDF)
Before this commit: robot arm, 10 links, 9 joints
Links:
- removed link left_gripper_base
- removed link left_gripper_finger
- removed link right_gripper_base
- removed link right_gripper_finger
Joints:
- removed joint l_g_base
- removed joint l_g_finger
- removed joint r_g_base
- removed joint r_g_finger

Commit message: Add files via upload

File: robot_arm/urdf/mybot.urdf (robot description, URDF)
Before this commit: robot arm, 6 links, 5 joints
Links:
- added link left_gripper_base, mass 0.01; collision box size=0.005 0.005 0.02; visual box size=0.005 0.005 0.02
- added link left_gripper_finger, mass 0.01; collision box size=0.008 0.008 0.05; visual box size=0.008 0.008 0.05
- added link right_gripper_base, mass 0.01; collision box size=0.005 0.005 0.02; visual box size=0.005 0.005 0.02
- added link right_gripper_finger, mass 0.01; collision box size=0.005 0.005 0.05; visual box size=0.008 0.008 0.05
Joints:
- added joint l_g_base: type revolute, parent hand, child left_gripper_base, origin xyz=0 0.02 0.035 rpy=-0.9162 0 0, axis 1 0 0, limit lower=0 upper=0.5236 effort=30.0 velocity=1.0
- added joint l_g_finger: type fixed, parent left_gripper_base, child left_gripper_finger, origin xyz=0 -0.01 0.03 rpy=0.3926 0 0
- added joint r_g_base: type revolute, parent hand, child right_gripper_base, origin xyz=0 -0.02 0.035 rpy=0.9162 0 0, axis 1 0 0, limit lower=-0.5236 upper=0 effort=100.0 velocity=1.0
- added joint r_g_finger: type fixed, parent right_gripper_base, child right_gripper_finger, origin xyz=0 0.01 0.03 rpy=-0.3926 0 0
- joint shoulder: limit lower=-1.5708 upper=0 effort=30.0 velocity=1.0 -> lower=-1.5708 upper=0.6981 effort=30.0 velocity=1.0
